Commit message: fix(hardware): add inertials to cosmetic URDF links + validation script
Add minimal inertial properties (0.05 kg) to LED strip and camera eye
links to prevent simulation instability. Create validate.py that parses
the URDF and reports links, joints, mass, limits, and structural issues.

Co-Authored-By: Claude Opus 4.6 <noreply@anthropic.com>

File: hardware/urdf/cleanwalker.urdf (robot description, URDF)
Before this commit: robot cleanwalker, 23 links, 22 joints
Links:
- link eye_left: mass None -> 0.05
- link eye_right: mass None -> 0.05
- link led_strip_left: mass None -> 0.05
- link led_strip_right: mass None -> 0.05
